File: Core/HI.sch (KiCad schematic (older format))
At the start: 17 parts, among them J4 Conn_01x10_Female, J8 Conn_01x10_Female, Q1 BSS84, Q10 BSS84, Q11 2N7002, Q12 2N7002, Q13 BSS84, Q2 BSS84, Q3 2N7002, Q4 BSS84, Q5 BSS84, Q6 2N7002, Q7 BSS84, Q8 2N7002, Q9 BSS84

Commit message: Add custom symbols and footprints
Parts:
- J4, J8: footprint CustomLib:PinSocket_1x10_P2.54mm_Vertical_SMD_Pin1Both -> Custom_FP:PinSocket_1x10_P2.54mm_Vertical_SMD_Pin1Both
- RV1: footprint CustomLib:VG039N -> Custom_FP:VG039N
Changed lines of the file:
@@
 F 0 "J8" H 10428 1276 50  0000 L CNN
 F 1 "Conn_01x10_Female" H 10428 1185 50  0000 L CNN
-F 2 "CustomLib:PinSocket_1x10_P2.54mm_Vertical_SMD_Pin1Both" H 10400 1300 50  0001 C CNN
+F 2 "Custom_FP:PinSocket_1x10_P2.54mm_Vertical_SMD_Pin1Both" H 10400 1300 50  0001 C CNN
 F 3 "~" H 10400 1300 50  0001 C CNN
 	1    10400 1300
@@
 F 0 "J4" H 10278 5026 50  0000 L CNN
 F 1 "Conn_01x10_Female" H 10278 4935 50  0000 L CNN
-F 2 "CustomLib:PinSocket_1x10_P2.54mm_Vertical_SMD_Pin1Both" H 10250 5050 50  0001 C CNN
+F 2 "Custom_FP:PinSocket_1x10_P2.54mm_Vertical_SMD_Pin1Both" H 10250 5050 50  0001 C CNN
 F 3 "~" H 10250 5050 50  0001 C CNN
 	1    10250 5050
@@
 F 0 "RV1" H 8980 3446 50  0000 R CNN
 F 1 "3k3" H 8980 3355 50  0000 R CNN
-F 2 "CustomLib:VG039N" H 9050 3400 50  0001 C CNN
+F 2 "Custom_FP:VG039N" H 9050 3400 50  0001 C CNN
 F 3 "~" H 9050 3400 50  0001 C CNN
 	1    9050 3400
