File: Core/MIDI_CV16.sch (KiCad schematic (older format))
At the start: 106 parts, among them J1 USB_C_Receptacle_USB2.0, J2 Conn_01x06_Male, J3 Conn_01x10_Female, J5 Conn_01x04, J7 Conn_01x10_Female, SW1 SW_Push_DPDT, U1 ATSAMD21G17D, U10 TL072, U11 TL072, U12 TL072, U13 MCP2517FD-xSL, U14 TLE9250V, U2 CD4052, U4 TL072, U5 TL072, U6 TL072, U7 TL072, U8 CD4052, U9 TL072, Y1 20MHz

Commit message: Update termination circuit
Parts:
- C49: value 22nF -> 4.7nF
- J1: symbol MIDI_CV16-rescue:USB_C_Receptacle_USB2.0-Connector -> Connector:USB_C_Receptacle_USB2.0
- R28, R59: value 120 -> 56
Other:
- note added: "31k"
- note added: "47k"
- note added: "91k"
- moved on the sheet: C11, C13, C14, C15, C17, C18, C19, C20, C21, C22, C23, C24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

Commit message: Add custom symbols and footprints
Parts:
- J1: footprint CustomLib:USB_C_Receptacle_GCT_USB4085_Slimmed -> Custom_FP:USB_C_Receptacle_GCT_USB4085_Slimmed
- J3, J7: footprint CustomLib:PinSocket_1x10_P2.54mm_Vertical_SMD_Pin1Both -> Custom_FP:PinSocket_1x10_P2.54mm_Vertical_SMD_Pin1Both
- J5: footprint CustomLib:MicroMatch_04_Vertical_SMD -> Custom_FP:MicroMatch_04_Vertical_SMD
- SW1: footprint CustomLib:SlideDPDT_JS202011 -> Custom_FP:SlideDPDT_JS202011
- Y1: footprint CustomLib:Crystal_2pin_2.0x2.5mm -> Custom_FP:Crystal_2pin_2.0x2.5mm
Changed lines of the file:
@@
 F 0 "J7" H 15228 4376 50  0000 L CNN
 F 1 "Conn_01x10_Female" H 15228 4285 50  0000 L CNN
-F 2 "CustomLib:PinSocket_1x10_P2.54mm_Vertical_SMD_Pin1Both" H 15200 4400 50  0001 C CNN
+F 2 "Custom_FP:PinSocket_1x10_P2.54mm_Vertical_SMD_Pin1Both" H 15200 4400 50  0001 C CNN
 F 3 "~" H 15200 4400 50  0001 C CNN
 	1    15200 4400
@@
 F 0 "J1" H 1607 10167 50  0000 C CNN
 F 1 "USB_C_Receptacle_USB2.0" H 1607 10076 50  0000 C CNN
-F 2 "CustomLib:USB_C_Receptacle_GCT_USB4085_Slimmed" H 1650 9300 50  0001 C CNN
+F 2 "Custom_FP:USB_C_Receptacle_GCT_USB4085_Slimmed" H 1650 9300 50  0001 C CNN
 F 3 "https://www.usb.org/sites/default/files/documents/usb_type-c.zip" H 1650 9300 50  0001 C CNN
 	1    1500 9300
@@
 F 0 "J3" H 9328 4426 50  0000 L CNN
 F 1 "Conn_01x10_Female" H 9328 4335 50  0000 L CNN
-F 2 "CustomLib:PinSocket_1x10_P2.54mm_Vertical_SMD_Pin1Both" H 9300 4450 50  0001 C CNN
+F 2 "Custom_FP:PinSocket_1x10_P2.54mm_Vertical_SMD_Pin1Both" H 9300 4450 50  0001 C CNN
 F 3 "~" H 9300 4450 50  0001 C CNN
 	1    9300 4450
@@
 F 0 "SW1" H 9000 9485 50  0000 C CNN
 F 1 "SW_Push_DPDT" H 9000 9394 50  0000 C CNN
-F 2 "CustomLib:SlideDPDT_JS202011" H 9000 9200 50  0001 C CNN
+F 2 "Custom_FP:SlideDPDT_JS202011" H 9000 9200 50  0001 C CNN
 F 3 "~" H 9000 9200 50  0001 C CNN
 	1    9000 9000
@@
 F 0 "J5" H 9780 10042 50  0000 L CNN
 F 1 "Conn_01x04" H 9780 9951 50  0000 L CNN
-F 2 "CustomLib:MicroMatch_04_Vertical_SMD" H 9700 10050 50  0001 C CNN
+F 2 "Custom_FP:MicroMatch_04_Vertical_SMD" H 9700 10050 50  0001 C CNN
 F 3 "~" H 9700 10050 50  0001 C CNN
 	1    9700 10050
@@
 F 0 "Y1" V 4704 10031 50  0000 L CNN
 F 1 "20MHz" V 4795 10031 50  0000 L CNN
-F 2 "CustomLib:Crystal_2pin_2.0x2.5mm" H 4750 9900 50  0001 C CNN
+F 2 "Custom_FP:Crystal_2pin_2.0x2.5mm" H 4750 9900 50  0001 C CNN
 F 3 "~" H 4750 9900 50  0001 C CNN
 	1    4750 9900
