File: Core/Powah.sch (KiCad schematic (older format))
At the start: 36 parts, among them J20 Conn_02x08_Odd_Even, U10 TL072, U11 TL072, U12 TL072, U3 MIC5504-3.3YM5, U4 TL072, U5 TL072, U6 TL072, U7 TL072, U9 TL072

Commit message: Add custom symbols and footprints
Parts:
- J20: footprint CustomLib:Header_2x8_Shrouded_SMD -> Custom_FP:Header_2x8_Shrouded_SMD
Changed lines of the file:
@@
 F 0 "J20" H 2500 2417 50  0000 C CNN
 F 1 "Conn_02x08_Odd_Even" H 2500 2326 50  0000 C CNN
-F 2 "CustomLib:Header_2x8_Shrouded_SMD" H 2450 1900 50  0001 C CNN
+F 2 "Custom_FP:Header_2x8_Shrouded_SMD" H 2450 1900 50  0001 C CNN
 F 3 "~" H 2450 1900 50  0001 C CNN
 	1    2450 1900
