File: Core/MIDI_CV16.kicad_sch (KiCad schematic)
At the start: 106 parts, among them J1 USB_C_Receptacle_USB2.0, J2 Conn_01x06_Male, J3 Conn_01x10_Female, J5 Conn_01x04, J7 Conn_01x10_Female, SW1 SW_Push_DPDT, U1 ATSAMD21G17D, U10 TL072, U11 TL072, U12 TL072, U13 MCP2517FD-xSL, U14 TLE9250V, U2 CD4052, U4 TL072, U5 TL072, U6 TL072, U7 TL072, U8 CD4052, U9 TL072, Y1 20MHz

Commit message: Fix DRC
Parts:
- R28, R59: value 56 -> 62
Connections:
- net MIDIBUS+ renamed M2IDI+
- net MIDIBUS- renamed M2IDI-
Changed lines of the file:
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@@
     )
   )
-  (global_label "MIDIBUS-" (shape bidirectional) (at 220.98 247.65 0)
+  (global_label "M2IDI-" (shape bidirectional) (at 220.98 247.65 0)
     (effects (font (size 1.27 1.27)) (justify left))
     (property "Intersheetrefs" "${INTERSHEET_REFS}" (at 220.98 247.65 0)
@@
     )
   )
-  (global_label "MIDIBUS+" (shape bidirectional) (at 220.98 242.57 0)
+  (global_label "M2IDI+" (shape bidirectional) (at 220.98 242.57 0)
     (effects (font (size 1.27 1.27)) (justify left))
     (property "Intersheetrefs" "${INTERSHEET_REFS}" (at 220.98 242.57 0)
@@
       (effects (font (size 1.27 1.27)))
     )
-    (property "Value" "56" (at 240.03 231.14 90)
+    (property "Value" "62" (at 240.03 231.14 90)
       (effects (font (size 1.27 1.27)))
     )
@@
       (effects (font (size 1.27 1.27)))
     )
-    (property "Value" "56" (at 240.03 220.98 90)
-      (effects (font (size 1.27 1.27)))
-    )
+    (property "Value" "62" (at 240.03 220.98 90)
+      (effects (font (size 1.27 1.27)))
+    )
