File: Core/MIDI_CV16.kicad_pcb (KiCad board)
At the start: 2 copper layers, 59.5 x 99.5 mm, 151 parts, among them J1 USB_C_Receptacle_USB2.0, J2 Conn_01x06_Male, J20 Conn_02x08_Odd_Even, J3 Conn_01x10_Female, J4 Conn_01x10_Female, J5 Conn_01x04, J7 Conn_01x10_Female, J8 Conn_01x10_Female, Q1 BSS84, Q10 BSS84, Q11 2N7002, Q12 2N7002, Q13 BSS84, Q2 BSS84, Q3 2N7002, Q4 BSS84, Q5 BSS84, Q6 2N7002, Q7 BSS84, Q8 2N7002, Q9 BSS84, SW1 SW_Push_DPDT, U1 ATSAMD21G15B-A, U10 TL072, U11 TL072, U12 TL072, U13 MCP2517FD-xSL, U14 TLE9250V, U2 CD4052, U3 MIC5504-3.3YM5, U4 TL072, U5 TL072, U6 TL072, U7 TL072, U8 CD4052, U9 TL072, Y1 20MHz

Commit message: Fix DRC errors
Parts:
- C49: value 22nF -> 4.7nF
- J1: footprint CustomLib:USB_C_Receptacle_GCT_USB4085_Slimmed -> Custom_FP:USB_C_Receptacle_GCT_USB4085_Slimmed
- J20: footprint CustomLib:Header_2x8_Shrouded_SMD -> Custom_FP:Header_2x8_Shrouded_SMD
- J3, J4, J7, J8: footprint CustomLib:PinSocket_1x10_P2.54mm_Vertical_SMD_Pin1Both -> Custom_FP:PinSocket_1x10_P2.54mm_Vertical_SMD_Pin1Both
- J5: footprint CustomLib:MicroMatch_04_Vertical_SMD -> Custom_FP:MicroMatch_04_Vertical_SMD
- R28, R59: value 120 -> 56
- RV1: footprint CustomLib:VG039N -> Custom_FP:VG039N
- SW1: footprint CustomLib:SlideDPDT_JS202011 -> Custom_FP:SlideDPDT_JS202011
- U1: value ATSAMD21G15B-A -> ATSAMD21G17D
- Y1: footprint CustomLib:Crystal_2pin_2.0x2.5mm -> Custom_FP:Crystal_2pin_2.0x2.5mm
- moved J2 2.00 mm to (101.8, 105.8), turned to 0 degrees
- moved R60 0.35 mm to (90.8, 103.0)
- moved C8 0.25 mm to (92.0, 102.0)
Routing:
- net SWCLK: track 26.3 -> 30.8 mm
- net SWDIO: track 22.4 -> 25.4 mm
- net +3V3: track 313.8 -> 311.4 mm, vias 27 -> 26
- net RESET: track 11.5 -> 13.5 mm

Commit message: Update to KiCAD 7
Other:
- net class Default removed

Commit message: Fix DRC
Parts:
- J1: footprint Custom_FP:USB_C_Receptacle_GCT_USB4085_Slimmed -> Connector_USB:USB_C_Receptacle_HRO_TYPE-C-31-M-12; moved to B.Cu
- R2, R3: moved to F.Cu
- moved J1 5.45 mm to (105.4, 94.6), turned to -90 degrees
- moved R3 4.47 mm to (101.2, 95.6)
- moved R2 4.07 mm to (101.2, 93.6), turned to 180 degrees
- moved Q13 0.35 mm to (76.5, 67.4)
- moved Q2 0.35 mm to (61.5, 67.4)
- moved Q5 0.35 mm to (66.5, 67.4)
- moved Q9 0.35 mm to (71.5, 67.4)
- moved C33 0.10 mm to (76.6, 94.2)
Connections:
- J1 pad A8: (no net) -> unconnected-(J1-SBU1-PadA8)
- J1 pad B8: (no net) -> unconnected-(J1-SBU2-PadB8)
- J2 pad 6: (no net) -> unconnected-(J2-Pin_6-Pad6)
- J20 pad 13: (no net) -> unconnected-(J20-Pin_13-Pad13)
- J20 pad 14: (no net) -> unconnected-(J20-Pin_14-Pad14)
- J20 pad 15: (no net) -> unconnected-(J20-Pin_15-Pad15)
- J20 pad 16: (no net) -> unconnected-(J20-Pin_16-Pad16)
- SW1 pad 3: (no net) -> unconnected-(SW1-C-Pad3)
- SW1 pad 6: (no net) -> unconnected-(SW1-C-Pad6)
- U1 pad 12: (no net) -> unconnected-(U1-PA07-Pad12)
- U1 pad 41: (no net) -> unconnected-(U1-PA28-Pad41)
- U1 pad 47: (no net) -> unconnected-(U1-PB02-Pad47)
- U1 pad 48: (no net) -> unconnected-(U1-PB03-Pad48)
- U1 pad 7: (no net) -> unconnected-(U1-PB08-Pad7)
- U1 pad 8: (no net) -> unconnected-(U1-PB09-Pad8)
- U13 pad 3: (no net) -> unconnected-(U13-CLKO/SOF-Pad3)
- U13 pad 8: (no net) -> unconnected-(U13-~{INT1}/GPIO1-Pad8)
- U13 pad 9: (no net) -> unconnected-(U13-~{INT0}/GPIO0/XSTBY-Pad9)
- U3 pad 4: (no net) -> unconnected-(U3-NC-Pad4)
Routing:
- net GND: track 70.1 -> 55.2 mm
- net USB_D-: track 14.9 -> 17.4 mm, vias 1 -> 2
- net Net-(J1-CC2): track 2.11 -> 4.28 mm, vias 0 -> 1
- net Net-(J1-SHIELD): track 19.3 -> 21.1 mm
- net Net-(J1-CC1): track 2.23 -> 3.98 mm, vias 0 -> 1
- net -VDC: track 161.2 -> 160.2 mm
- net USB_D+: track 15.3 -> 16.2 mm, vias 1 -> 2
- net VBUS: track 12.4 -> 11.6 mm, vias 0 -> 1

Commit message: Fix more DRC
Parts:
- R28, R59: value 56 -> 62
Connections:
- net MIDIBUS+ renamed M2IDI+
- net MIDIBUS- renamed M2IDI-
Changed lines of the file:
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@@
   (net 101 "MUX_B")
   (net 102 "MUX_A")
-  (net 103 "MIDIBUS+")
-  (net 104 "MIDIBUS-")
+  (net 103 "M2IDI-")
+  (net 104 "M2IDI+")
   (net 105 "Net-(U6B--)")
   (net 106 "Net-(U7A--)")
@@
         (effects (font (size 1 1) (thickness 0.15)))
     )
-    (fp_text value "56" (at 0 1.43) (layer "F.Fab")
+    (fp_text value "62" (at 0 1.43) (layer "F.Fab")
         (effects (font (size 1 1) (thickness 0.15)))
     )
@@
         (effects (font (size 1 1) (thickness 0.15)))
     )
-    (fp_text value "56" (at 0 1.43) (layer "F.Fab")
+    (fp_text value "62" (at 0 1.43) (layer "F.Fab")
         (effects (font (size 1 1) (thickness 0.15)))
     )
@@
       (net 18 "+3V3") (pinfunction "VIO") (pintype "power_in"))
     (pad "6" smd roundrect (at 2.625 0.635) (size 1.65 0.6) (layers "F.Cu" "F.Paste" "F.Mask") (roundrect_rratio 0.25)
-      (net 104 "MIDIBUS-") (pinfunction "CANL") (pintype "bidirectional"))
+      (net 103 "M2IDI-") (pinfunction "CANL") (pintype "bidirectional"))
     (pad "7" smd roundrect (at 2.625 -0.635) (size 1.65 0.6) (layers "F.Cu" "F.Paste" "F.Mask") (roundrect_rratio 0.25)
-      (net 103 "MIDIBUS+") (pinfunction "CANH") (pintype "bidirectional"))
+      (net 104 "M2IDI+") (pinfunction "CANH") (pintype "bidirectional"))
     (pad "8" smd roundrect (at 2.625 -1.905) (size 1.65 0.6) (layers "F.Cu" "F.Paste" "F.Mask") (roundrect_rratio 0.25)
       (net 1 "GND") (pinfunction "S") (pintype "input"))
@@
       (net 109 "Net-(R28-Pad2)") (pinfunction "A") (pintype "passive"))
     (pad "2" smd roundrect (at -2.75 0 270) (size 2.5 1.2) (layers "B.Cu" "B.Paste" "B.Mask") (roundrect_rratio 0.25)
-      (net 103 "MIDIBUS+") (pinfunction "B") (pintype "passive"))
+      (net 104 "M2IDI+") (pinfunction "B") (pintype "passive"))
     (pad "3" smd roundrect (at -2.75 -2.5 270) (size 2.5 1.2) (layers "B.Cu" "B.Paste" "B.Mask") (roundrect_rratio 0.25)
       (net 126 "unconnected-(SW1-C-Pad3)") (pinfunction "C") (pintype "passive+no_connect"))
@@
       (net 110 "Net-(R59-Pad2)") (pinfunction "A") (pintype "passive"))
     (pad "5" smd roundrect (at 2.75 0 270) (size 2.5 1.2) (layers "B.Cu" "B.Paste" "B.Mask") (roundrect_rratio 0.25)
-      (net 104 "MIDIBUS-") (pinfunction "B") (pintype "passive"))
+      (net 103 "M2IDI-") (pinfunction "B") (pintype "passive"))
     (pad "6" smd roundrect (at 2.75 -2.5 270) (size 2.5 1.2) (layers "B.Cu" "B.Paste" "B.Mask") (roundrect_rratio 0.25)
       (net 127 "unconnected-(SW1-C-Pad6)") (pinfunction "C") (pintype "passive+no_connect"))
@@
       (net 23 "Net-(J5-Pin_1)") (pinfunction "Pin_1") (pintype "passive"))
     (pad "2" smd rect (at 0.635 2.35 270) (size 1.5 3.5) (layers "B.Cu" "B.Paste" "B.Mask")
-      (net 104 "MIDIBUS-") (pinfunction "Pin_2") (pintype "passive"))
+      (net 103 "M2IDI-") (pinfunction "Pin_2") (pintype "passive"))
     (pad "3" smd rect (at -0.635 -2.35 270) (size 1.5 3.5) (layers "B.Cu" "B.Paste" "B.Mask")
-      (net 103 "MIDIBUS+") (pinfunction "Pin_3") (pintype "passive"))
+      (net 104 "M2IDI+") (pinfunction "Pin_3") (pintype "passive"))
     (pad "4" smd rect (at -1.905 2.35 270) (size 1.5 3.5) (layers "B.Cu" "B.Paste" "B.Mask")
       (net 23 "Net-(J5-Pin_1)") (pinfunction "Pin_4") (pintype "passive"))
@@
   (segment (start 65.806795 137.306795) (end 67.35358 135.76001) (width 0.25) (layer "B.Cu") (net 102))
   (segment (start 79.09998 123.440608) (end 79.09998 119.75) (width 0.25) (layer "B.Cu") (net 102))
-  (segment (start 88.854 55.525) (end 89.154 55.225) (width 0.2) (layer "F.Cu") (net 103))
-  (segment (start 85.535 55.525) (end 88.854 55.525) (width 0.2) (layer "F.Cu") (net 103))
-  (segment (start 85.125 55.115) (end 85.535 55.525) (width 0.2) (layer "F.Cu") (net 103))
-  (via (at 89.154 55.225) (size 0.8) (drill 0.4) (layers "F.Cu" "B.Cu") (net 103))
-  (segment (start 106.6 55.115) (end 104.635 55.115) (width 0.2) (layer "B.Cu") (net 103))
-  (segment (start 89.154 55.225) (end 89.454 55.525) (width 0.2) (layer "B.Cu") (net 103))
-  (segment (start 93 53) (end 93 54.5) (width 0.2) (layer "B.Cu") (net 103))
-  (segment (start 98.5 55.525) (end 93 55.525) (width 0.2) (layer "B.Cu") (net 103))
-  (segment (start 98.91 55.115) (end 98.5 55.525) (width 0.2) (layer "B.Cu") (net 103))
-  (segment (start 93 55.525) (end 92.482 55.525) (width 0.2) (layer "B.Cu") (net 103))
-  (segment (start 104.635 55.115) (end 98.91 55.115) (width 0.2) (layer "B.Cu") (net 103))
-  (segment (start 89.454 55.525) (end 92.482 55.525) (width 0.2) (layer "B.Cu") (net 103))
-  (segment (start 93 54.5) (end 93 55.525) (width 0.2) (layer "B.Cu") (net 103))
-  (segment (start 88.854 55.975) (end 89.154 56.275) (width 0.2) (layer "F.Cu") (net 104))
-  (segment (start 85.535 55.975) (end 88.854 55.975) (width 0.2) (layer "F.Cu") (net 104))
-  (segment (start 85.125 56.385) (end 85.535 55.975) (width 0.2) (layer "F.Cu") (net 104))
-  (via (at 89.154 56.275) (size 0.8) (drill 0.4) (layers "F.Cu" "B.Cu") (net 104))
-  (segment (start 93 55.975) (end 92.488 55.975) (width 0.2) (layer "B.Cu") (net 104))
-  (segment (start 89.454 55.975) (end 92.488 55.975) (width 0.2) (layer "B.Cu") (net 104))
-  (segment (start 98.5 55.975) (end 93 55.975) (width 0.2) (layer "B.Cu") (net 104))
-  (segment (start 89.154 56.275) (end 89.454 55.975) (width 0.2) (layer "B.Cu") (net 104))
-  (segment (start 93 57) (end 93 55.975) (width 0.2) (layer "B.Cu") (net 104))
-  (segment (start 99.885 56.385) (end 98.91 56.385) (width 0.2) (layer "B.Cu") (net 104))
-  (segment (start 101.9 56.385) (end 99.885 56.385) (width 0.2) (layer "B.Cu") (net 104))
-  (segment (start 93 58.5) (end 93 57) (width 0.2) (layer "B.Cu") (net 104))
-  (segment (start 98.91 56.385) (end 98.5 55.975) (width 0.2) (layer "B.Cu") (net 104))
+  (segment (start 88.854 55.975) (end 89.154 56.275) (width 0.2) (layer "F.Cu") (net 103))
+  (segment (start 85.535 55.975) (end 88.854 55.975) (width 0.2) (layer "F.Cu") (net 103))
+  (segment (start 85.125 56.385) (end 85.535 55.975) (width 0.2) (layer "F.Cu") (net 103))
+  (via (at 89.154 56.275) (size 0.8) (drill 0.4) (layers "F.Cu" "B.Cu") (net 103))
+  (segment (start 93 55.975) (end 92.488 55.975) (width 0.2) (layer "B.Cu") (net 103))
+  (segment (start 89.454 55.975) (end 92.488 55.975) (width 0.2) (layer "B.Cu") (net 103))
+  (segment (start 98.5 55.975) (end 93 55.975) (width 0.2) (layer "B.Cu") (net 103))
+  (segment (start 89.154 56.275) (end 89.454 55.975) (width 0.2) (layer "B.Cu") (net 103))
+  (segment (start 93 57) (end 93 55.975) (width 0.2) (layer "B.Cu") (net 103))
+  (segment (start 99.885 56.385) (end 98.91 56.385) (width 0.2) (layer "B.Cu") (net 103))
+  (segment (start 101.9 56.385) (end 99.885 56.385) (width 0.2) (layer "B.Cu") (net 103))
+  (segment (start 93 58.5) (end 93 57) (width 0.2) (layer "B.Cu") (net 103))
+  (segment (start 98.91 56.385) (end 98.5 55.975) (width 0.2) (layer "B.Cu") (net 103))
+  (segment (start 88.854 55.525) (end 89.154 55.225) (width 0.2) (layer "F.Cu") (net 104))
+  (segment (start 85.535 55.525) (end 88.854 55.525) (width 0.2) (layer "F.Cu") (net 104))
+  (segment (start 85.125 55.115) (end 85.535 55.525) (width 0.2) (layer "F.Cu") (net 104))
+  (via (at 89.154 55.225) (size 0.8) (drill 0.4) (layers "F.Cu" "B.Cu") (net 104))
+  (segment (start 106.6 55.115) (end 104.635 55.115) (width 0.2) (layer "B.Cu") (net 104))
+  (segment (start 89.154 55.225) (end 89.454 55.525) (width 0.2) (layer "B.Cu") (net 104))
+  (segment (start 93 53) (end 93 54.5) (width 0.2) (layer "B.Cu") (net 104))
+  (segment (start 98.5 55.525) (end 93 55.525) (width 0.2) (layer "B.Cu") (net 104))
+  (segment (start 98.91 55.115) (end 98.5 55.525) (width 0.2) (layer "B.Cu") (net 104))
+  (segment (start 93 55.525) (end 92.482 55.525) (width 0.2) (layer "B.Cu") (net 104))
+  (segment (start 104.635 55.115) (end 98.91 55.115) (width 0.2) (layer "B.Cu") (net 104))
+  (segment (start 89.454 55.525) (end 92.482 55.525) (width 0.2) (layer "B.Cu") (net 104))
+  (segment (start 93 54.5) (end 93 55.525) (width 0.2) (layer "B.Cu") (net 104))
   (segment (start 70.135 127.1525) (end 70.5375 126.75) (width 0.25) (layer "F.Cu") (net 105))
   (segment (start 70.5375 126.75) (end 70.5375 123.825) (width 0.25) (layer "F.Cu") (net 105))
