File: Core/MIDI_CV16.kicad_pcb (KiCad board)
At the start: 2 copper layers, 59.5 x 99.5 mm, 167 parts, among them J1 USB_C_Receptacle_USB2.0, J2 Conn_01x06_Male, J20 Conn_02x08_Odd_Even, J3 Conn_01x10_Female, J4 Conn_01x10_Female, J5 Conn_01x04, J7 Conn_01x10_Female, J8 Conn_01x10_Female, Q1 BSS84, Q10 BSS84, Q11 2N7002, Q12 2N7002, Q13 BSS84, Q14 2N7002, Q15 ZXMP3A13FTA, Q16 ZXMP3A13FTA, Q17 PMV88ENER, Q2 BSS84, Q3 2N7002, Q4 BSS84, Q5 BSS84, Q6 2N7002, Q7 BSS84, Q8 2N7002, Q9 BSS84, SW1 SW_Push_DPDT, SW2 SW_SPST, SW3 SW_SPST, U1 RP2040, U10 TL072, U11 TL072, U12 TL072, U13 MCP2517FD-xSL, U14 MCP2562FD-ESN, U15 MAX5134, U16 CAT25640, U17 IS25LP032D, U2 TMUX4052, U3 MIC5504-3.3YM5, U4 TL072, U5 TL072, U6 TL072, U7 TL072, U8 TMUX4052, U9 TL072, Y1 20MHz, Y2 ECS-120-18-33-JGN-TR3

Commit message: Fix DRC warnings
Routing:
- net +VDC: track 269.5 -> 266.7 mm
- net -VDC: track 169.4 -> 167.3 mm
- net Net-(U13-OSC2): track 5.45 -> 3.89 mm
- net Net-(U13-OSC1): track 5.45 -> 3.89 mm
- net +3V3: track 222.7 -> 221.2 mm
- net GND: track 26.1 -> 24.6 mm
- net +5V: track 351.7 -> 350.9 mm
- net RESET: track 49.4 -> 48.6 mm
- net Net-(U4B--): track 4.46 -> 3.93 mm
- net Net-(U9A--): track 4.48 -> 3.96 mm
- net Net-(U7A--): track 4.48 -> 3.96 mm
- net Net-(U6A--): track 4.48 -> 3.96 mm
- net Net-(U5A--): track 4.48 -> 3.96 mm
- net Net-(U4A--): track 4.47 -> 3.94 mm
- net Net-(U11A--): track 4.48 -> 3.96 mm
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
Commit message: Fix more drc warnings........
Routing:
- net GND: track 24.6 -> 27.9 mm
Changed lines of the file:
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@@
   (segment (start 80.525 111.5125) (end 80.525 112.725) (width 0.25) (layer "B.Cu") (net 1))
   (segment (start 77.275 118.475) (end 77.275 118.975) (width 0.25) (layer "B.Cu") (net 1))
+  (segment (start 87.268629 93.5) (end 85.75 95.018629) (width 0.25) (layer "B.Cu") (net 1))
   (segment (start 80.525 108.425) (end 79.95 107.85) (width 0.25) (layer "B.Cu") (net 1))
   (segment (start 85.4 98) (end 85.4 99.4) (width 0.2) (layer "B.Cu") (net 1))
+  (segment (start 85.75 95.018629) (end 85.75 95.5) (width 0.25) (layer "B.Cu") (net 1))
+  (segment (start 85.75 95.5) (end 86.198744 95.948744) (width 0.25) (layer "B.Cu") (net 1))
   (segment (start 85.545056 96.637786) (end 87.282842 94.9) (width 0.2) (layer "B.Cu") (net 1))
   (segment (start 82.75 112.85) (end 82.82 112.85) (width 0.25) (layer "B.Cu") (net 1))

Commit message: Finalize module
Parts:
- C27, C28: value 3.3µF -> 10µF; footprint Capacitor_Tantalum_SMD:CP_EIA-3216-18_Kemet-A -> Capacitor_SMD:C_0805_2012Metric
- R28, R59, R63, R8: footprint Resistor_SMD:R_0603_1608Metric -> Resistor_SMD:R_0805_2012Metric
- U2, U8: value TMUX4052 -> MC74LVXT4052
- moved C27 0.61 mm to (73.8, 98.5)
- moved R8 0.60 mm to (57.2, 62.0)
- moved R28 0.35 mm to (91.8, 54.8)
- moved R59 0.35 mm to (91.8, 56.8)
- moved C28 0.35 mm to (73.0, 108.8)
- moved R63 0.25 mm to (56.5, 64.8)
- moved C25 0.10 mm to (60.8, 130.0)
Other:
- rule pad_to_mask_clearance: 0.05 -> 0
- board text added: "M2IDI_CV16 V3.0 GuavTek"
- board text removed: "MIDIBUS_CV16 V3.0 GuavTek"

Commit message: Layout v3.1
Parts:
- added R10: 470, Resistor_SMD:R_0603_1608Metric, F.Cu at (75.0, 138.8)
- added R12: 470, Resistor_SMD:R_0603_1608Metric, F.Cu at (76.0, 125.8)
- added R14: 470, Resistor_SMD:R_0603_1608Metric, F.Cu at (84.0, 138.8)
- added R16: 470, Resistor_SMD:R_0603_1608Metric, F.Cu at (85.0, 125.8)
- C11, C13, C14, C15, C17, C18, C19, C20, C21, C22, C23, C24, C4, C6, C7, C9: value 100pF -> 1.5nF NP0; moved to B.Cu
- C25, C26, C66, C67: moved to F.Cu
- C29, C30, C31, C32, C34, C35, C36, C37, C38, C39, C40, C41, C42, C43, C44, C45, R11, R13, R15, R17, R19, R21, R23, R25, R26, R27, R29, R30, R31, R32, R35, R37, R39, R41, R43, R45, R47, R49, R51, R52, R53, R54, R55, R56, R57, R58, R7, R9, U10, U11, U12, U4, U5, U6, U7, U9: moved to B.Cu
- SW2, SW3: footprint Custom_FP:Tactile_angled_5x5.4_SMD -> Custom_FP:Tactile_angled_SPST_5x5.4_SMD
- U2, U8: value MC74LVXT4052 -> TMUX1309; footprint Package_SO:SOIC-16_3.9x9.9mm_P1.27mm -> Package_SO:TSSOP-16_4.4x5mm_P0.65mm; moved to F.Cu
- moved C67 46.5 mm to (56.5, 145.2)
- moved C58 35.2 mm to (90.2, 122.8), turned to 180 degrees
- moved C37 27.4 mm to (57.4, 119.7), turned to 0 degrees
- moved C14 25.3 mm to (57.4, 121.2), turned to 180 degrees
- moved C29 24.4 mm to (68.1, 145.7), turned to 0 degrees
- moved C65 23.5 mm to (104.2, 121.0), turned to 0 degrees
- moved R19 23.2 mm to (57.4, 122.7), turned to 180 degrees
- moved C66 22.4 mm to (73.8, 143.8), turned to 90 degrees
- moved R25 22.3 mm to (68.1, 144.2), turned to 0 degrees
- moved C38 21.3 mm to (102.7, 123.9), turned to 0 degrees
- moved R31 21.1 mm to (57.4, 124.2), turned to 180 degrees
- moved SW3 20.8 mm to (55.1, 85.5)
- moved R9 20.2 mm to (68.1, 142.7), turned to 0 degrees
- moved R52 20.0 mm to (102.7, 122.4), turned to 0 degrees
- moved C44 19.7 mm to (102.7, 145.8), turned to 0 degrees
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Connections:
- U1 pad 11: SPI_MISO -> MUX_A
- U1 pad 12: EEPROM_CS -> MUX_B
- U1 pad 13: SPI_SCK -> MUX_INH
- U1 pad 14: SPI_MOSI -> DAC_MOSI
- U1 pad 15: LEDC1 -> DAC_SCK
- U1 pad 16: LEDC2 -> DAC_CS
- U1 pad 17: LEDC3 -> LEDC1
- U1 pad 18: LEDC4 -> unconnected-(U1-GPIO15-Pad18)
- U1 pad 27: LEDR5 -> LEDC2
- U1 pad 28: LEDC5 -> LEDC3
- U1 pad 29: LEDC6 -> LEDC4
- U1 pad 30: LEDC7 -> LEDR5
- U1 pad 31: CAN_MISO -> LEDC5
- U1 pad 32: CAN_CS -> LEDC6
- U1 pad 34: CAN_SCK -> LEDC7
- U1 pad 35: CAN_MOSI -> LEDC8
- U1 pad 37: LEDC8 -> CAN_CS
- U1 pad 5: unconnected-(U1-GPIO3-Pad5) -> EEPROM_CS
- U1 pad 6: MUX_B -> SPI_MISO
- U1 pad 7: MUX_A -> unconnected-(U1-GPIO5-Pad7)
- U1 pad 8: MUX_INH -> SPI_SCK
- U1 pad 9: DAC_CS -> SPI_MOSI
- U13 pad 10: CAN_SCK -> SPI_SCK
- U13 pad 11: CAN_MOSI -> SPI_MOSI
- U13 pad 12: CAN_MISO -> SPI_MISO
- U15 pad 10: SPI_SCK -> DAC_SCK
- U15 pad 8: SPI_MOSI -> DAC_MOSI
- U2 pad 13: Net-(U15-OUT0) -> Net-(U2-X)
- U2 pad 3: Net-(U15-OUT1) -> Net-(U2-Y)
- U8 pad 13: Net-(U15-OUT2) -> Net-(U8-X)
- U8 pad 3: Net-(U15-OUT3) -> Net-(U8-Y)
Routing:
- net +VDC: track 266.7 -> 171.4 mm, vias 30 -> 13
- net MUX_INH: track 131.5 -> 61.3 mm, vias 0 -> 5
- net MUX_A: track 105.8 -> 59.8 mm, vias 0 -> 5
- net SPI_MISO: track 18.7 -> 62.5 mm, vias 2 -> 3
- net MUX_B: track 105.7 -> 62.3 mm, vias 0 -> 5
- net DAC_SCK: track 0.00 -> 30.1 mm, vias 0 -> 2
- net SPI_MOSI: track 31.5 -> 60.8 mm, vias 2 -> 3
- net CAN_MISO: track 29.2 -> 0.00 mm, vias 2 -> 0
- net CAN_SCK: track 27.5 -> 0.00 mm, vias 2 -> 0
- net -VDC: track 167.3 -> 140.9 mm
- net CAN_MOSI: track 26.3 -> 0.00 mm, vias 2 -> 0
- net DAC_MOSI: track 0.00 -> 20.8 mm, vias 0 -> 2
- net Net-(U15-OUT1): track 26.3 -> 9.11 mm, vias 0 -> 1
- net Net-(U11A-+): track 7.69 -> 24.6 mm
- net Net-(U2-X2): track 7.42 -> 24.2 mm
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Other:
- board text added: "M2IDI_CV16 V3.1 GuavTek"
- board text removed: "M2IDI_CV16 V3.0 GuavTek"
