File: Front/MIDI_CV16_Front.kicad_pcb (KiCad board)
At the start: 2 copper layers, 59.5 x 128.5 mm, 23 parts, among them J1 Screw_Terminal_01x01, J10 Conn_01x01, J11 Conn_01x01, J12 Conn_01x01, J13 Conn_01x01, J14 Conn_01x01, J15 Conn_01x01, J16 Conn_01x01, J17 Conn_01x01, J18 Conn_01x01, J19 Conn_01x01, J2 Screw_Terminal_01x01, J20 Conn_01x01, J21 Conn_01x01, J22 Conn_01x01, J23 Conn_01x01, J3 Screw_Terminal_01x01, J4 Screw_Terminal_01x01, J5 Conn_01x01, J6 Conn_01x01, J7 Conn_01x01, J8 Conn_01x01, J9 Conn_01x01

Commit message: Maybe actually fix drc
Parts:
- J12, J13, J14, J15, J16, J17, J18, J19, J20, J21, J22, J23, J6, J7, J8, J9: footprint MountingHole:MountingHole_6.2mm_M6 -> Custom_FP:JackHole_3.5mm
Connections:
- J1 pad 1: Net-(J1-Pad1) -> unconnected-(J1-Pin_1-Pad1)
- J2 pad 1: Net-(J2-Pad1) -> unconnected-(J2-Pin_1-Pad1)
- J3 pad 1: Net-(J3-Pad1) -> unconnected-(J3-Pin_1-Pad1)
- J4 pad 1: Net-(J4-Pad1) -> unconnected-(J4-Pin_1-Pad1)
