File: Front/MIDI_CV16_Front.kicad_sch (KiCad schematic)
At the start: 23 parts, among them J1 Screw_Terminal_01x01, J10 Conn_01x01, J11 Conn_01x01, J12 Conn_01x01, J13 Conn_01x01, J14 Conn_01x01, J15 Conn_01x01, J16 Conn_01x01, J17 Conn_01x01, J18 Conn_01x01, J19 Conn_01x01, J2 Screw_Terminal_01x01, J20 Conn_01x01, J21 Conn_01x01, J22 Conn_01x01, J23 Conn_01x01, J3 Screw_Terminal_01x01, J4 Screw_Terminal_01x01, J5 Conn_01x01, J6 Conn_01x01, J7 Conn_01x01, J8 Conn_01x01, J9 Conn_01x01

Commit message: Update to KiCAD 7
Other:
- company: (none) -> GuavTek
- title: (none) -> M2IDI - CV16 FRONT
Changed lines of the file:
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@@
 (kicad_sch (version 20230121) (generator eeschema)
   (paper "A3")
+  (title_block
+    (title "M2IDI - CV16 FRONT")
+    (date "2023-04-19")
+    (rev "3.0")
+    (company "GuavTek")
+  )
   (junction (at 220.98 59.69) (diameter 0) (color 0 0 0 0)
   )

Commit message: Fix front panel DRC
Parts:
- J12, J13, J14, J15, J16, J17, J18, J19, J20, J21, J22, J23, J6, J7, J8, J9: footprint MountingHole:MountingHole_6.2mm_M6 -> MountingHole:MountingHole_6.4mm_M6
Changed lines of the file:
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@@
       (effects (font (size 1.27 1.27)) (justify left))
     )
-    (property "Footprint" "MountingHole:MountingHole_6.2mm_M6" (at 146.05 49.53 0)
+    (property "Footprint" "MountingHole:MountingHole_6.4mm_M6" (at 146.05 49.53 0)
       (effects (font (size 1.27 1.27)) hide)
     )
@@
       (effects (font (size 1.27 1.27)) (justify left))
     )
-    (property "Footprint" "MountingHole:MountingHole_6.2mm_M6" (at 146.05 54.61 0)
+    (property "Footprint" "MountingHole:MountingHole_6.4mm_M6" (at 146.05 54.61 0)
       (effects (font (size 1.27 1.27)) hide)
     )
@@
       (effects (font (size 1.27 1.27)) (justify left))
     )
-    (property "Footprint" "MountingHole:MountingHole_6.2mm_M6" (at 146.05 59.69 0)
+    (property "Footprint" "MountingHole:MountingHole_6.4mm_M6" (at 146.05 59.69 0)
       (effects (font (size 1.27 1.27)) hide)
     )
@@
       (effects (font (size 1.27 1.27)) (justify left))
     )
-    (property "Footprint" "MountingHole:MountingHole_6.2mm_M6" (at 146.05 64.77 0)
+    (property "Footprint" "MountingHole:MountingHole_6.4mm_M6" (at 146.05 64.77 0)
       (effects (font (size 1.27 1.27)) hide)
     )
@@
       (effects (font (size 1.27 1.27)) (justify left))
     )
-    (property "Footprint" "MountingHole:MountingHole_6.2mm_M6" (at 173.99 49.53 0)
+    (property "Footprint" "MountingHole:MountingHole_6.4mm_M6" (at 173.99 49.53 0)
       (effects (font (size 1.27 1.27)) hide)
     )
@@
       (effects (font (size 1.27 1.27)) (justify left))
     )
-    (property "Footprint" "MountingHole:MountingHole_6.2mm_M6" (at 173.99 54.61 0)
+    (property "Footprint" "MountingHole:MountingHole_6.4mm_M6" (at 173.99 54.61 0)
       (effects (font (size 1.27 1.27)) hide)
     )
@@
       (effects (font (size 1.27 1.27)) (justify left))
     )
-    (property "Footprint" "MountingHole:MountingHole_6.2mm_M6" (at 173.99 59.69 0)
+    (property "Footprint" "MountingHole:MountingHole_6.4mm_M6" (at 173.99 59.69 0)
       (effects (font (size 1.27 1.27)) hide)
     )
@@
       (effects (font (size 1.27 1.27)) (justify left))
     )
-    (property "Footprint" "MountingHole:MountingHole_6.2mm_M6" (at 173.99 64.77 0)
+    (property "Footprint" "MountingHole:MountingHole_6.4mm_M6" (at 173.99 64.77 0)
       (effects (font (size 1.27 1.27)) hide)
     )
@@
       (effects (font (size 1.27 1.27)) (justify left))
     )
-    (property "Footprint" "MountingHole:MountingHole_6.2mm_M6" (at 200.66 49.53 0)
+    (property "Footprint" "MountingHole:MountingHole_6.4mm_M6" (at 200.66 49.53 0)
       (effects (font (size 1.27 1.27)) hide)
     )
@@
       (effects (font (size 1.27 1.27)) (justify left))
     )
-    (property "Footprint" "MountingHole:MountingHole_6.2mm_M6" (at 200.66 54.61 0)
+    (property "Footprint" "MountingHole:MountingHole_6.4mm_M6" (at 200.66 54.61 0)
       (effects (font (size 1.27 1.27)) hide)
     )
@@
       (effects (font (size 1.27 1.27)) (justify left))
     )
-    (property "Footprint" "MountingHole:MountingHole_6.2mm_M6" (at 200.66 59.69 0)
+    (property "Footprint" "MountingHole:MountingHole_6.4mm_M6" (at 200.66 59.69 0)
       (effects (font (size 1.27 1.27)) hide)
     )
@@
       (effects (font (size 1.27 1.27)) (justify left))
     )
-    (property "Footprint" "MountingHole:MountingHole_6.2mm_M6" (at 200.66 64.77 0)
+    (property "Footprint" "MountingHole:MountingHole_6.4mm_M6" (at 200.66 64.77 0)
       (effects (font (size 1.27 1.27)) hide)
     )
@@
       (effects (font (size 1.27 1.27)) (justify left))
     )
-    (property "Footprint" "MountingHole:MountingHole_6.2mm_M6" (at 228.6 49.53 0)
+    (property "Footprint" "MountingHole:MountingHole_6.4mm_M6" (at 228.6 49.53 0)
       (effects (font (size 1.27 1.27)) hide)
     )
@@
       (effects (font (size 1.27 1.27)) (justify left))
     )
-    (property "Footprint" "MountingHole:MountingHole_6.2mm_M6" (at 228.6 54.61 0)
+    (property "Footprint" "MountingHole:MountingHole_6.4mm_M6" (at 228.6 54.61 0)
       (effects (font (size 1.27 1.27)) hide)
     )
@@
       (effects (font (size 1.27 1.27)) (justify left))
     )
-    (property "Footprint" "MountingHole:MountingHole_6.2mm_M6" (at 228.6 59.69 0)
+    (property "Footprint" "MountingHole:MountingHole_6.4mm_M6" (at 228.6 59.69 0)
       (effects (font (size 1.27 1.27)) hide)
     )
@@
       (effects (font (size 1.27 1.27)) (justify left))
     )
-    (property "Footprint" "MountingHole:MountingHole_6.2mm_M6" (at 228.6 64.77 0)
-      (effects (font (size 1.27 1.27)) hide)
-    )
+    (property "Footprint" "MountingHole:MountingHole_6.4mm_M6" (at 228.6 64.77 0)
+      (effects (font (size 1.27 1.27)) hide)
+    )

Commit message: Maybe actually fix drc
Parts:
- J12, J13, J14, J15, J16, J17, J18, J19, J20, J21, J22, J23, J6, J7, J8, J9: footprint MountingHole:MountingHole_6.4mm_M6 -> Custom_FP:JackHole_3.5mm
Changed lines of the file:
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@@
       (effects (font (size 1.27 1.27)) (justify left))
     )
-    (property "Footprint" "MountingHole:MountingHole_6.4mm_M6" (at 146.05 49.53 0)
+    (property "Footprint" "Custom_FP:JackHole_3.5mm" (at 146.05 49.53 0)
       (effects (font (size 1.27 1.27)) hide)
     )
@@
       (effects (font (size 1.27 1.27)) (justify left))
     )
-    (property "Footprint" "MountingHole:MountingHole_6.4mm_M6" (at 146.05 54.61 0)
+    (property "Footprint" "Custom_FP:JackHole_3.5mm" (at 146.05 54.61 0)
       (effects (font (size 1.27 1.27)) hide)
     )
@@
       (effects (font (size 1.27 1.27)) (justify left))
     )
-    (property "Footprint" "MountingHole:MountingHole_6.4mm_M6" (at 146.05 59.69 0)
+    (property "Footprint" "Custom_FP:JackHole_3.5mm" (at 146.05 59.69 0)
       (effects (font (size 1.27 1.27)) hide)
     )
@@
       (effects (font (size 1.27 1.27)) (justify left))
     )
-    (property "Footprint" "MountingHole:MountingHole_6.4mm_M6" (at 146.05 64.77 0)
+    (property "Footprint" "Custom_FP:JackHole_3.5mm" (at 146.05 64.77 0)
       (effects (font (size 1.27 1.27)) hide)
     )
@@
       (effects (font (size 1.27 1.27)) (justify left))
     )
-    (property "Footprint" "MountingHole:MountingHole_6.4mm_M6" (at 173.99 49.53 0)
+    (property "Footprint" "Custom_FP:JackHole_3.5mm" (at 173.99 49.53 0)
       (effects (font (size 1.27 1.27)) hide)
     )
@@
       (effects (font (size 1.27 1.27)) (justify left))
     )
-    (property "Footprint" "MountingHole:MountingHole_6.4mm_M6" (at 173.99 54.61 0)
+    (property "Footprint" "Custom_FP:JackHole_3.5mm" (at 173.99 54.61 0)
       (effects (font (size 1.27 1.27)) hide)
     )
@@
       (effects (font (size 1.27 1.27)) (justify left))
     )
-    (property "Footprint" "MountingHole:MountingHole_6.4mm_M6" (at 173.99 59.69 0)
+    (property "Footprint" "Custom_FP:JackHole_3.5mm" (at 173.99 59.69 0)
       (effects (font (size 1.27 1.27)) hide)
     )
@@
       (effects (font (size 1.27 1.27)) (justify left))
     )
-    (property "Footprint" "MountingHole:MountingHole_6.4mm_M6" (at 173.99 64.77 0)
+    (property "Footprint" "Custom_FP:JackHole_3.5mm" (at 173.99 64.77 0)
       (effects (font (size 1.27 1.27)) hide)
     )
@@
       (effects (font (size 1.27 1.27)) (justify left))
     )
-    (property "Footprint" "MountingHole:MountingHole_6.4mm_M6" (at 200.66 49.53 0)
+    (property "Footprint" "Custom_FP:JackHole_3.5mm" (at 200.66 49.53 0)
       (effects (font (size 1.27 1.27)) hide)
     )
@@
       (effects (font (size 1.27 1.27)) (justify left))
     )
-    (property "Footprint" "MountingHole:MountingHole_6.4mm_M6" (at 200.66 54.61 0)
+    (property "Footprint" "Custom_FP:JackHole_3.5mm" (at 200.66 54.61 0)
       (effects (font (size 1.27 1.27)) hide)
     )
@@
       (effects (font (size 1.27 1.27)) (justify left))
     )
-    (property "Footprint" "MountingHole:MountingHole_6.4mm_M6" (at 200.66 59.69 0)
+    (property "Footprint" "Custom_FP:JackHole_3.5mm" (at 200.66 59.69 0)
       (effects (font (size 1.27 1.27)) hide)
     )
@@
       (effects (font (size 1.27 1.27)) (justify left))
     )
-    (property "Footprint" "MountingHole:MountingHole_6.4mm_M6" (at 200.66 64.77 0)
+    (property "Footprint" "Custom_FP:JackHole_3.5mm" (at 200.66 64.77 0)
       (effects (font (size 1.27 1.27)) hide)
     )
@@
       (effects (font (size 1.27 1.27)) (justify left))
     )
-    (property "Footprint" "MountingHole:MountingHole_6.4mm_M6" (at 228.6 49.53 0)
+    (property "Footprint" "Custom_FP:JackHole_3.5mm" (at 228.6 49.53 0)
       (effects (font (size 1.27 1.27)) hide)
     )
@@
       (effects (font (size 1.27 1.27)) (justify left))
     )
-    (property "Footprint" "MountingHole:MountingHole_6.4mm_M6" (at 228.6 54.61 0)
+    (property "Footprint" "Custom_FP:JackHole_3.5mm" (at 228.6 54.61 0)
       (effects (font (size 1.27 1.27)) hide)
     )
@@
       (effects (font (size 1.27 1.27)) (justify left))
     )
-    (property "Footprint" "MountingHole:MountingHole_6.4mm_M6" (at 228.6 59.69 0)
+    (property "Footprint" "Custom_FP:JackHole_3.5mm" (at 228.6 59.69 0)
       (effects (font (size 1.27 1.27)) hide)
     )
@@
       (effects (font (size 1.27 1.27)) (justify left))
     )
-    (property "Footprint" "MountingHole:MountingHole_6.4mm_M6" (at 228.6 64.77 0)
-      (effects (font (size 1.27 1.27)) hide)
-    )
+    (property "Footprint" "Custom_FP:JackHole_3.5mm" (at 228.6 64.77 0)
+      (effects (font (size 1.27 1.27)) hide)
+    )
