File: IO/MIDI_CV16_IO.sch (KiCad schematic (older format))
At the start: 111 parts, among them J1 Conn_01x10_Male, J10 AudioJack2_SwitchT, J11 Conn_01x10_Male, J12 AudioJack2_SwitchT, J13 AudioJack2_SwitchT, J14 AudioJack2_SwitchT, J15 AudioJack2_SwitchT, J16 AudioJack2_SwitchT, J17 AudioJack2_SwitchT, J18 AudioJack2_SwitchT, J19 AudioJack2_SwitchT, J2 Conn_01x10_Male, J20 Conn_01x10_Male, J3 AudioJack2_SwitchT, J4 AudioJack2_SwitchT, J5 AudioJack2_SwitchT, J6 AudioJack2_SwitchT, J7 AudioJack2_SwitchT, J8 AudioJack2_SwitchT, J9 AudioJack2_SwitchT, SW1 SW_SPST, SW2 SW_SPST, SW3 SW_SPST

Commit message: Add custom symbols and footprints
Parts:
- D1, D2, D21, D22, D23, D24, D25, D26, D27, D28, D29, D3, D30, D31, D32, D33, D34, D35, D36, D37, D38, D39, D4, D40, D41, D42, D43, D44, D45, D46, D47, D48, D49, D50, D51, D52, D53, D54, D55, D56: footprint LED_THT:LED_D3.0mm -> Custom_FP:LED_D3.0mm_NoCourtyard
- J10, J12, J13, J14, J15, J16, J17, J18, J19, J3, J4, J5, J6, J7, J8, J9: footprint CustomLib:PJ398SM -> Custom_FP:PJ398SM
